Commit message: attempted fix

File: moveo_urdf/urdf/moveo_urdf_newer.urdf (robot description, URDF)
Before this commit: robot moveo_urdf, 12 links, 11 joints
Links:
- added link odom, mass 8.0643
Joints:
- added joint odom_joint: type fixed, parent base_link, child odom, origin xyz=0 0 0 rpy=0 0 0
- joint Joint_1: origin xyz=0 -0.2425 .13 rpy=1.5708 9.5417E-17 2.7766 -> xyz=0 -0.2425 0 rpy=1.5708 9.5417E-17 2.7766
- joint Pivot_Arm_Gripper_Idol_Joint: mimic (none) -> joint=Gripper_Idol_Gear_Joint multiplier=1 offset=0
- joint Pivot_Arm_Gripper_Servo_Joint: mimic (none) -> joint=Gripper_Servo_Gear_Joint multiplier=1 offset=0
- joint Tip_Gripper_Idol_Joint: mimic (none) -> joint=Gripper_Idol_Gear_Joint multiplier=-1 offset=0
- joint Tip_Gripper_Servo_Joint: mimic (none) -> joint=Gripper_Servo_Gear_Joint multiplier=1 offset=0
