Commit message: Renamed files

File: moveo_industrial_experimental/moveo6_meshes/BCN3D/BCN3D.urdf (robot description, URDF)
Before this commit: robot BCN3D, 8 links, 7 joints
Links:
- link base_link: geometry collision mesh filename=package://moveo6_meshes/moveo6/bin_stl/base_link_m-binary.s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; visual mesh filename=package://moveo6_meshes/moveo6/bin_stl/base_link_m-binary.s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
- link moveo_1_1: geometry collision mesh filename=package://moveo6_meshes/moveo6/bin_stl/moveo_1_1_m-binary.s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; visual mesh filename=package://moveo6_meshes/moveo6/bin_stl/moveo_1_1_m-binary.s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
- link moveo_2_1: geometry collision mesh filename=package://moveo6_meshes/moveo6/bin_stl/moveo_2_1_m-binary.s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; visual mesh filename=package://moveo6_meshes/moveo6/bin_stl/moveo_2_1_m-binary.s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
- link moveo_3_1: geometry collision mesh filename=package://moveo6_meshes/moveo6/bin_stl/moveo_3_1_m-binary.s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; visual mesh filename=package://moveo6_meshes/moveo6/bin_stl/moveo_3_1_m-binary.s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
- link moveo_4_1: geometry collision mesh filename=package://moveo6_meshes/moveo6/bin_stl/moveo_4_1_m-binary.s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; visual mesh filename=package://moveo6_meshes/moveo6/bin_stl/moveo_4_1_m-binary.s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
- link moveo_5_1: geometry collision mesh filename=package://moveo6_meshes/moveo6/bin_stl/moveo_5_1_m-binary.s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; visual mesh filename=package://moveo6_meshes/moveo6/bin_stl/moveo_5_1_m-binary.s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
- link moveo_6_1: geometry collision mesh filename=package://moveo6_meshes/moveo6/bin_stl/moveo_6_1_m-binary.s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; visual mesh filename=package://moveo6_meshes/moveo6/bin_stl/moveo_6_1_m-binary.s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
- link moveo_7_1: geometry collision mesh filename=package://moveo6_meshes/moveo6/bin_stl/moveo_7_1_m-binary.s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; visual mesh filename=package://moveo6_meshes/moveo6/bin_stl/moveo_7_1_m-binary.s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
